File: BoardA2.sch (EAGLE design)
At the start: 15 parts, among them J1 FEMALE 2x3, T1 2N2222

Commit message: Update 2
Connections:
- new net DC-CTRL: J1.2
- net 5V: now also J1.6; no longer J1.2
- net ADC-CH1: now also J1.5; no longer J1.6
Changed lines of the file:
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@@
 </segment>
 <segment>
-<pinref part="J1" gate="G$1" pin="2"/>
-<junction x="43.18" y="71.12"/>
-<label x="45.72" y="71.12" size="1.778" layer="95"/>
+<pinref part="J1" gate="G$1" pin="6"/>
+<junction x="43.18" y="66.04"/>
+<label x="43.18" y="66.04" size="1.016" layer="95" xref="yes"/>
 </segment>
 </net>
@@
 </segment>
 <segment>
-<pinref part="J1" gate="G$1" pin="6"/>
-<junction x="43.18" y="66.04"/>
-<label x="45.72" y="66.04" size="1.778" layer="95"/>
+<pinref part="J1" gate="G$1" pin="5"/>
+<junction x="27.94" y="66.04"/>
+<label x="27.94" y="66.04" size="1.016" layer="95" rot="R180" xref="yes"/>
 </segment>
 </net>
@@
 <pinref part="J1" gate="G$1" pin="4"/>
 <junction x="43.18" y="68.58"/>
-<label x="45.72" y="68.58" size="1.778" layer="95"/>
+<label x="43.18" y="68.58" size="1.016" layer="95" xref="yes"/>
 </segment>
 </net>
@@
 </segment>
 </net>
+<net name="DC-CTRL" class="0">
+<segment>
+<pinref part="J1" gate="G$1" pin="2"/>
+<junction x="43.18" y="71.12"/>
+<label x="43.18" y="71.12" size="1.016" layer="95" xref="yes"/>
+</segment>
+</net>

Commit message: Mid board Rerouting 1
Work in progress. Please do not commit any changes to Board2
Connections:
- removed net ADC-SLK: TEENSY1-12.5
- removed net N$11: ADC.4
- removed net TEENSY1: TEENSY1-12.1
- net ADC-SCLK: now also TEENSY1-12.5
Changed lines of the file:
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@@
 <junction x="-12.7" y="48.26"/>
+</segment>
+<segment>
+<pinref part="TEENSY1-12" gate="G$1" pin="5"/>
+<junction x="-88.9" y="63.5"/>
+<label x="-88.9" y="63.5" size="0.762" layer="95" xref="yes"/>
 </segment>
 </net>
 <net name="ADC-CONVST" class="0">
 <segment>
-<pinref part="ADC" gate="G$1" pin="5"/>
-<label x="-12.7" y="53.34" size="0.762" layer="95" rot="R180" xref="yes"/>
-<junction x="-12.7" y="53.34"/>
-</segment>
-<segment>
 <junction x="-88.9" y="55.88"/>
 <label x="-88.9" y="55.88" size="0.762" layer="95" xref="yes"/>
 </segment>
-</net>
-<net name="N$11" class="0">
 <segment>
-<pinref part="ADC" gate="G$1" pin="4"/>
-<wire x1="-12.7" y1="55.88" x2="-15.24" y2="55.88" width="0.1524" layer="91"/>
+<pinref part="ADC" gate="G$1" pin="5"/>
+<junction x="-12.7" y="53.34"/>
+<label x="-12.7" y="53.34" size="1.016" layer="95" rot="R180" xref="yes"/>
 </segment>
 </net>
@@
 <junction x="-88.9" y="66.04"/>
 <label x="-88.9" y="66.04" size="0.762" layer="95" xref="yes"/>
-</segment>
-</net>
-<net name="TEENSY1" class="0">
-<segment>
-<pinref part="TEENSY1-12" gate="G$1" pin="1"/>
-<junction x="-88.9" y="53.34"/>
 </segment>
 </net>
@@
 </segment>
 </net>
-<net name="ADC-SLK" class="0">
-<segment>
-<pinref part="TEENSY1-12" gate="G$1" pin="5"/>
-<junction x="-88.9" y="63.5"/>
-<label x="-88.9" y="63.5" size="0.762" layer="95" xref="yes"/>
-</segment>
-</net>

Commit message: Board2 Missing signal
Connections:
- removed net ADC-CONVST: ADC.5
- new net ADC-CON: ADC.5, TEENSY1-12.2
Changed lines of the file:
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@@
-</segment>
-</net>
-<net name="ADC-CONVST" class="0">
-<segment>
-<junction x="-88.9" y="55.88"/>
-<label x="-88.9" y="55.88" size="0.762" layer="95" xref="yes"/>
-</segment>
-<segment>
-<pinref part="ADC" gate="G$1" pin="5"/>
-<junction x="-12.7" y="53.34"/>
-<label x="-12.7" y="53.34" size="1.016" layer="95" rot="R180" xref="yes"/>
 </segment>
 </net>
@@
 </segment>
 </net>
+<net name="ADC-CON" class="0">
+<segment>
+<pinref part="ADC" gate="G$1" pin="5"/>
+<junction x="-12.7" y="53.34"/>
+<label x="-12.7" y="53.34" size="1.016" layer="95" rot="R180" xref="yes"/>
+</segment>
+<segment>
+<pinref part="TEENSY1-12" gate="G$1" pin="2"/>
+<junction x="-88.9" y="55.88"/>
+<label x="-88.9" y="55.88" size="0.762" layer="95" xref="yes"/>
+</segment>
+</net>
