File: BoardA2.sch (EAGLE design)
At the start: 15 parts, among them J1 FEMALE 2x3, T1 2N2222

Commit message: routing
Parts:
- C1: device SparkFun-Capacitors:0.1UF-50V-20%(PTH)KIT-EZ -> capacitor-wima:C5/2.5
- C2: device SparkFun-Passives:CAPPTH2 -> capacitor-wima:C5/2.5
- D1: value 1N4004 -> (none); device diode:1N4004 -> eagle-ltspice:DIODE_E-DO35-7
Other:
- moved on the sheet: C1, C2
Changed lines of the file:
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@@
 <part name="OSCILLATOR" library="Smartcrutches" deviceset="CLOCK-ECS-100X" device=""/>
 <part name="ADC" library="Smartcrutches" deviceset="DIL24" device="-3" value="AD7890-10"/>
-<part name="C1" library="SparkFun-Capacitors" deviceset="0.1UF-50V-20%(PTH)" device="KIT-EZ" value="0.1 uf"/>
+<part name="C1" library="capacitor-wima" library_urn="urn:adsk.eagle:library:116" deviceset="C" device="5/2.5" value="0.1 uf"/>
 <part name="J1" library="SparkFun-Connectors" deviceset="CONN_03X2" device="FEMALE" value="FEMALE 2x3"/>
 <part name="IMU" library="Smartcrutches" deviceset="IMU" device="" value="TSS-EM/3Space"/>
@@
 <part name="R2" library="resistor" library_urn="urn:adsk.eagle:library:348" deviceset="R-US_" device="0204/5" value="10kohm"/>
 <part name="T1" library="transistor" library_urn="urn:adsk.eagle:library:402" deviceset="2N2222" device=""/>
-<part name="D1" library="diode" library_urn="urn:adsk.eagle:library:210" deviceset="1N4004" device=""/>
-<part name="C2" library="SparkFun-Passives" deviceset="CAP" device="PTH2" value="0.1uf"/>
+<part name="D1" library="eagle-ltspice" library_urn="urn:adsk.eagle:library:217" deviceset="DIODE_E-" device="DO35-7"/>
+<part name="C2" library="capacitor-wima" library_urn="urn:adsk.eagle:library:116" deviceset="C" device="5/2.5" value="0.1uf"/>
 <part name="MOTOR" library="SparkFun-Connectors" deviceset="CONN_02" device=""/>
 <part name="LOWERLOADCELL" library="SparkFun-Connectors" deviceset="CONN_05" device=""/>
@@
 <instance part="R2" gate="G$1" x="71.12" y="71.12" rot="R90"/>
 <instance part="T1" gate="G$1" x="76.2" y="78.74"/>
-<instance part="D1" gate="1" x="78.74" y="91.44" rot="R90"/>
+<instance part="D1" gate="G$1" x="78.74" y="91.44" rot="R90"/>
 <instance part="C2" gate="G$1" x="86.36" y="88.9"/>
 <instance part="MOTOR" gate="G$1" x="60.96" y="93.98"/>
@@
 </segment>
 <segment>
-<pinref part="D1" gate="1" pin="C"/>
-<wire x1="78.74" y1="93.98" x2="78.74" y2="96.52" width="0.1524" layer="91"/>
+<pinref part="D1" gate="G$1" pin="C"/>
+<wire x1="76.2" y1="91.44" x2="78.74" y2="96.52" width="0.1524" layer="91"/>
 <wire x1="78.74" y1="96.52" x2="86.36" y2="96.52" width="0.1524" layer="91"/>
 <pinref part="C2" gate="G$1" pin="1"/>
-<wire x1="86.36" y1="96.52" x2="86.36" y2="93.98" width="0.1524" layer="91"/>
+<wire x1="86.36" y1="96.52" x2="86.36" y2="91.44" width="0.1524" layer="91"/>
 <junction x="86.36" y="96.52"/>
 <wire x1="86.36" y1="96.52" x2="86.36" y2="99.06" width="0.1524" layer="91"/>
@@
 <pinref part="ADC" gate="G$1" pin="15"/>
 <pinref part="C1" gate="G$1" pin="1"/>
-<wire x1="2.54" y1="40.64" x2="5.08" y2="40.64" width="0.1524" layer="91"/>
+<wire x1="2.54" y1="40.64" x2="7.62" y2="40.64" width="0.1524" layer="91"/>
 <junction x="2.54" y="40.64"/>
 </segment>
@@
 <pinref part="ADC" gate="G$1" pin="24"/>
 <wire x1="2.54" y1="63.5" x2="12.7" y2="63.5" width="0.1524" layer="91"/>
-<wire x1="12.7" y1="63.5" x2="12.7" y2="40.64" width="0.1524" layer="91"/>
+<wire x1="12.7" y1="63.5" x2="15.24" y2="40.64" width="0.1524" layer="91"/>
 <pinref part="C1" gate="G$1" pin="2"/>
-<wire x1="12.7" y1="40.64" x2="15.24" y2="40.64" width="0.1524" layer="91"/>
 <label x="15.24" y="40.64" size="1.778" layer="95" xref="yes"/>
 </segment>
@@
 <pinref part="C2" gate="G$1" pin="2"/>
 <wire x1="78.74" y1="83.82" x2="86.36" y2="83.82" width="0.1524" layer="91"/>
-<wire x1="86.36" y1="83.82" x2="86.36" y2="86.36" width="0.1524" layer="91"/>
-<pinref part="D1" gate="1" pin="A"/>
-<wire x1="78.74" y1="88.9" x2="78.74" y2="83.82" width="0.1524" layer="91"/>
+<pinref part="D1" gate="G$1" pin="A"/>
+<wire x1="81.28" y1="91.44" x2="78.74" y2="83.82" width="0.1524" layer="91"/>
 <junction x="78.74" y="83.82"/>
 <wire x1="78.74" y1="83.82" x2="73.66" y2="83.82" width="0.1524" layer="91"/>

Commit message: cosmetic changes
Connections:
- net E+ renamed AMP-E+
- net N$10 renamed AMP-SD
- net N$4 renamed ADC-CLK
- net N$5 renamed AMP-E-
- net N$7 renamed AMP-A-
- net N$9 renamed AMP-A+
- net 5V: now also D1.A; no longer D1.C
- net N$6: now also D1.C; no longer D1.A
Other:
- moved on the sheet: C1, D1
Changed lines of the file:
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@@
 <instance part="OSCILLATOR" gate="G$1" x="-48.26" y="48.26"/>
 <instance part="ADC" gate="G$1" x="-5.08" y="48.26"/>
-<instance part="C1" gate="G$1" x="10.16" y="40.64" rot="R90"/>
+<instance part="C1" gate="G$1" x="7.62" y="40.64" rot="R90"/>
 <instance part="J1" gate="G$1" x="35.56" y="68.58"/>
 <instance part="IMU" gate="G$1" x="-7.62" y="83.82"/>
@@
 <instance part="R2" gate="G$1" x="71.12" y="71.12" rot="R90"/>
 <instance part="T1" gate="G$1" x="76.2" y="78.74"/>
-<instance part="D1" gate="G$1" x="78.74" y="91.44" rot="R90"/>
+<instance part="D1" gate="G$1" x="78.74" y="91.44" rot="R180"/>
 <instance part="C2" gate="G$1" x="86.36" y="88.9"/>
 <instance part="MOTOR" gate="G$1" x="60.96" y="93.98"/>
@@
 </segment>
 <segment>
-<pinref part="D1" gate="G$1" pin="C"/>
-<wire x1="76.2" y1="91.44" x2="78.74" y2="96.52" width="0.1524" layer="91"/>
-<wire x1="78.74" y1="96.52" x2="86.36" y2="96.52" width="0.1524" layer="91"/>
 <pinref part="C2" gate="G$1" pin="1"/>
 <wire x1="86.36" y1="96.52" x2="86.36" y2="91.44" width="0.1524" layer="91"/>
@@
 <wire x1="86.36" y1="96.52" x2="86.36" y2="99.06" width="0.1524" layer="91"/>
 <label x="86.36" y="99.06" size="1.778" layer="95" rot="R90" xref="yes"/>
+<pinref part="MOTOR" gate="G$1" pin="2"/>
+<wire x1="86.36" y1="96.52" x2="78.74" y2="96.52" width="0.1524" layer="91"/>
+<pinref part="D1" gate="G$1" pin="A"/>
+<wire x1="78.74" y1="96.52" x2="68.58" y2="96.52" width="0.1524" layer="91"/>
+<wire x1="78.74" y1="93.98" x2="78.74" y2="96.52" width="0.1524" layer="91"/>
 <junction x="78.74" y="96.52"/>
-<pinref part="MOTOR" gate="G$1" pin="2"/>
-<wire x1="78.74" y1="96.52" x2="68.58" y2="96.52" width="0.1524" layer="91"/>
 </segment>
 <segment>
@@
 <pinref part="ADC" gate="G$1" pin="15"/>
 <pinref part="C1" gate="G$1" pin="1"/>
-<wire x1="2.54" y1="40.64" x2="7.62" y2="40.64" width="0.1524" layer="91"/>
+<wire x1="2.54" y1="40.64" x2="5.08" y2="40.64" width="0.1524" layer="91"/>
 <junction x="2.54" y="40.64"/>
 </segment>
@@
 <pinref part="ADC" gate="G$1" pin="24"/>
 <wire x1="2.54" y1="63.5" x2="12.7" y2="63.5" width="0.1524" layer="91"/>
-<wire x1="12.7" y1="63.5" x2="15.24" y2="40.64" width="0.1524" layer="91"/>
+<wire x1="12.7" y1="63.5" x2="12.7" y2="40.64" width="0.1524" layer="91"/>
 <pinref part="C1" gate="G$1" pin="2"/>
-<label x="15.24" y="40.64" size="1.778" layer="95" xref="yes"/>
+<label x="12.7" y="40.64" size="1.778" layer="95" xref="yes"/>
 </segment>
 <segment>
@@
 </segment>
 </net>
-<net name="N$4" class="0">
+<net name="ADC-CLK" class="0">
 <segment>
 <pinref part="OSCILLATOR" gate="G$1" pin="OUT"/>
@@
 <pinref part="C2" gate="G$1" pin="2"/>
 <wire x1="78.74" y1="83.82" x2="86.36" y2="83.82" width="0.1524" layer="91"/>
-<pinref part="D1" gate="G$1" pin="A"/>
-<wire x1="81.28" y1="91.44" x2="78.74" y2="83.82" width="0.1524" layer="91"/>
 <junction x="78.74" y="83.82"/>
 <wire x1="78.74" y1="83.82" x2="73.66" y2="83.82" width="0.1524" layer="91"/>
@@
 <pinref part="MOTOR" gate="G$1" pin="1"/>
 <wire x1="73.66" y1="93.98" x2="68.58" y2="93.98" width="0.1524" layer="91"/>
+<pinref part="D1" gate="G$1" pin="C"/>
+<wire x1="78.74" y1="83.82" x2="78.74" y2="88.9" width="0.1524" layer="91"/>
 </segment>
 </net>
@@
 </segment>
 </net>
-<net name="E+" class="0">
+<net name="AMP-E+" class="0">
 <segment>
 <pinref part="LOADCELL_AMP" gate="G$1" pin="E+"/>
@@
 </segment>
 </net>
-<net name="N$5" class="0">
+<net name="AMP-E-" class="0">
 <segment>
 <pinref part="LOADCELL_AMP" gate="G$1" pin="E-"/>
@@
 </segment>
 </net>
-<net name="N$7" class="0">
+<net name="AMP-A-" class="0">
 <segment>
 <pinref part="LOADCELL_AMP" gate="G$1" pin="A-"/>
@@
 </segment>
 </net>
-<net name="N$9" class="0">
+<net name="AMP-A+" class="0">
 <segment>
 <pinref part="LOADCELL_AMP" gate="G$1" pin="A+"/>
@@
 </segment>
 </net>
-<net name="N$10" class="0">
+<net name="AMP-SD" class="0">
 <segment>
 <pinref part="LOADCELL_AMP" gate="G$1" pin="SD"/>

Commit message: update
Parts:
- IMU: value TSS-EM/3Space -> TSS-EM
Changed lines of the file:
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@@
 <part name="C1" library="capacitor-wima" library_urn="urn:adsk.eagle:library:116" deviceset="C" device="5/2.5" value="0.1 uf"/>
 <part name="J1" library="SparkFun-Connectors" deviceset="CONN_03X2" device="FEMALE" value="FEMALE 2x3"/>
-<part name="IMU" library="Smartcrutches" deviceset="IMU" device="" value="TSS-EM/3Space"/>
+<part name="IMU" library="Smartcrutches" deviceset="IMU" device="" value="TSS-EM"/>
 <part name="LOADCELL_AMP" library="Smartcrutches" deviceset="LOADCELLAMP" device="" value="HX711"/>
 <part name="TEENSY1-12" library="SparkFun-Connectors" deviceset="CONN_12" device=""/>
@@
 <junction x="2.54" y="55.88"/>
 <junction x="2.54" y="58.42"/>
-<junction x="2.54" y="60.96"/>
 <label x="2.54" y="55.88" size="1.778" layer="95" xref="yes"/>
 <junction x="2.54" y="50.8"/>
@@
 <label x="-12.7" y="35.56" size="1.016" layer="95" rot="R180" xref="yes"/>
 <junction x="-12.7" y="35.56"/>
-</segment>
-<segment>
-<pinref part="ADC" gate="G$1" pin="2"/>
-<junction x="-12.7" y="60.96"/>
-<label x="-12.7" y="60.96" size="1.016" layer="95" rot="R180" xref="yes"/>
 </segment>
 <segment>
@@
 <label x="43.18" y="66.04" size="1.016" layer="95" xref="yes"/>
 </segment>
+<segment>
+<pinref part="ADC" gate="G$1" pin="2"/>
+<junction x="-12.7" y="60.96"/>
+<label x="-12.7" y="60.96" size="1.016" layer="95" rot="R180" xref="yes"/>
+</segment>
 </net>
