File: BoardA2.brd (EAGLE design)
At the start: 44 x 93 mm, 18 parts, among them J1 FEMALE 2x3, T1 2N2222

Commit message: routing
Parts:
- C1: device SparkFun-Capacitors:CAP-PTH-SMALL-KIT -> capacitor-wima:C5B2.5
- C2: device SparkFun-Passives:CAP-PTH-SMALL2 -> capacitor-wima:C5B2.5
- D1: value 1N4004 -> (none); device diode:DO41-10 -> eagle-ltspice:DIODE_DO35-7
- moved C2 12.6 mm to (36.7, 77.0)
- moved T1 10.2 mm to (29.0, 77.5), turned to 270 degrees
- moved D1 4.52 mm to (37.4, 71.6)
- moved C1 1.69 mm to (15.2, 9.62)
- moved IMU 0.51 mm to (20.7, 15.0)
- turned R1 to 90 degrees
Connections:
- net 5V: now also D1.A; no longer D1.C
- net N$6: now also D1.C; no longer D1.A
Routing:
- net MOTOR: track 0.00 -> 74.2 mm
- net 5V: track 86.3 -> 151.0 mm
- net N$6: track 31.2 -> 0.00 mm
- net ADC-DIN: track 0.00 -> 24.7 mm
- net ADC-DOUT: track 0.00 -> 23.9 mm
- net ADC-CON: track 19.8 -> 41.3 mm, vias 0 -> 1
- net N$8: track 11.8 -> 0.00 mm
- net GND: track 91.1 -> 100.2 mm
- net ADC-SCLK: track 7.66 -> 0.00 mm
- net IMU-TX: track 0.00 -> 2.46 mm

Commit message: final changes
Parts:
- moved C1 5.66 mm to (20.8, 10.5), turned to 0 degrees
- moved MOTOR 1.30 mm to (19.9, 89.3)
- moved R2 1.25 mm to (24.1, 83.4)
- moved R1 0.85 mm to (20.6, 83.4)
- moved T1 0.77 mm to (28.9, 78.3), turned to 0 degrees
- turned D1 to 0 degrees
Routing:
- net 5V: track 151.0 -> 242.0 mm
- net GND: track 100.2 -> 189.3 mm, vias 0 -> 2
- net IMU-RX: track 0.00 -> 75.3 mm
- net IMU-TX: track 2.46 -> 75.0 mm
- net ADC-SCLK: track 0.00 -> 45.2 mm, vias 0 -> 1
- net N$4: track 0.00 -> 36.8 mm
- net N$6: track 0.00 -> 34.8 mm
- net ADC-TFS: track 0.00 -> 34.2 mm
- net ADC-CH2: track 0.00 -> 26.4 mm, vias 0 -> 1
- net ADC-CH1: track 0.00 -> 24.4 mm, vias 0 -> 1
- net N$8: track 0.00 -> 16.5 mm
- net N$3: track 0.00 -> 12.9 mm
- net ADC-RFS: track 0.00 -> 11.9 mm

Commit message: last update
Routing:
- net 5V: track 242.0 -> 246.1 mm
Changed lines of the file:
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@@
 <wire x1="11.287" y1="41.465" x2="18.907" y2="41.465" width="1.27" layer="16"/>
 <wire x1="31.958621875" y1="65.16725" x2="31.958621875" y2="63.454621875" width="1.27" layer="1"/>
-<wire x1="31.958621875" y1="63.454621875" x2="31.115" y2="62.611" width="1.27" layer="1"/>
-<wire x1="31.115" y1="62.611" x2="28.448" y2="59.944" width="1.27" layer="1"/>
-<wire x1="28.448" y1="59.944" x2="25.908" y2="59.944" width="1.27" layer="1"/>
-<wire x1="25.908" y1="59.944" x2="14.097" y2="59.944" width="1.27" layer="1"/>
+<wire x1="31.0515" y1="62.5475" x2="31.958621875" y2="63.454621875" width="1.27" layer="1"/>
+<wire x1="31.0515" y1="62.5475" x2="28.448" y2="59.944" width="1.27" layer="1"/>
+<wire x1="28.448" y1="59.944" x2="14.097" y2="59.944" width="1.27" layer="1"/>
 <wire x1="14.097" y1="59.944" x2="10.033" y2="55.88" width="1.27" layer="1"/>
 <wire x1="10.033" y1="55.88" x2="10.033" y2="49.553" width="1.27" layer="1"/>
@@
 <wire x1="37.25" y1="4.26" x2="38.677" y2="4.26" width="1.27" layer="1"/>
 <wire x1="41.656" y1="28.321" x2="41.656" y2="7.239" width="1.27" layer="1"/>
-<wire x1="41.656" y1="28.321" x2="41.021" y2="28.956" width="1.27" layer="1"/>
-<wire x1="40.386" y1="29.591" x2="41.021" y2="28.956" width="1.27" layer="1"/>
-<wire x1="40.386" y1="29.591" x2="36.83" y2="29.591" width="1.27" layer="1"/>
-<wire x1="36.83" y1="29.591" x2="27.432" y2="29.591" width="1.27" layer="1"/>
+<wire x1="40.386" y1="29.591" x2="41.656" y2="28.321" width="1.27" layer="1"/>
+<wire x1="40.386" y1="29.591" x2="27.432" y2="29.591" width="1.27" layer="1"/>
 <wire x1="27.432" y1="29.591" x2="25.908" y2="31.115" width="1.27" layer="1"/>
 <wire x1="25.908" y1="31.115" x2="25.908" y2="37.827" width="1.27" layer="1"/>
@@
 <wire x1="22.987" y1="41.529" x2="18.971" y2="41.529" width="1.27" layer="1"/>
 <wire x1="18.971" y1="41.529" x2="18.907" y2="41.465" width="1.27" layer="1"/>
-<wire x1="31.115" y1="62.611" x2="32.258" y2="62.611" width="1.27" layer="1"/>
-<wire x1="32.258" y1="62.611" x2="40.767" y2="54.102" width="1.27" layer="1"/>
-<wire x1="40.767" y1="54.102" x2="40.767" y2="50.447678125" width="1.27" layer="1"/>
-<wire x1="40.767" y1="50.447678125" x2="40.793603125" y2="50.4208875" width="1.27" layer="1"/>
+<wire x1="40.793603125" y1="50.4208875" x2="40.767" y2="50.447678125" width="1.27" layer="1"/>
 <wire x1="40.793603125" y1="50.4208875" x2="40.789940625" y2="49.37176875" width="1.27" layer="1"/>
 <wire x1="40.789940625" y1="49.37176875" x2="40.789940625" y2="28.806059375" width="1.27" layer="1"/>
 <wire x1="40.789940625" y1="28.806059375" x2="41.148" y2="28.448" width="1.27" layer="1"/>
-<wire x1="41.021" y1="28.956" x2="40.789940625" y2="28.806059375" width="0" layer="19" extent="1-1"/>
+<wire x1="40.767" y1="61.087" x2="39.497" y2="62.357" width="1.27" layer="1"/>
+<wire x1="40.767" y1="50.447678125" x2="40.767" y2="61.087" width="1.27" layer="1"/>
+<wire x1="39.497" y1="62.357" x2="31.242" y2="62.357" width="1.27" layer="1"/>
+<wire x1="31.242" y1="62.357" x2="31.0515" y2="62.5475" width="1.27" layer="1"/>
+<wire x1="41.656" y1="28.321" x2="41.148" y2="28.448" width="0" layer="19" extent="1-1"/>
 </signal>
 <signal name="N$1">

Commit message: cosmetic changes
Parts:
- moved C1 0.63 mm to (20.8, 11.1)
- turned D1 to 180 degrees
Connections:
- net E+ renamed AMP-E+
- net N$10 renamed AMP-SD
- net N$4 renamed ADC-CLK
- net N$5 renamed AMP-E-
- net N$7 renamed AMP-A-
- net N$9 renamed AMP-A+
- net 5V: now also D1.C; no longer D1.A
- net N$6: now also D1.A; no longer D1.C
Routing:
- net 5V: track 246.1 -> 240.4 mm
- net IMU-TX: track 75.0 -> 78.9 mm
- net IMU-RX: track 75.3 -> 77.3 mm
- net ADC-CH2: track 26.4 -> 28.0 mm
- net ADC-CH1: track 24.4 -> 25.8 mm
- net AMP-A-: track 13.1 -> 14.5 mm
- net GND: track 189.3 -> 188.1 mm, vias 2 -> 0
- net AMP-SD: track 12.5 -> 11.6 mm
- net N$3: track 12.9 -> 13.6 mm

Commit message: update
Parts:
- IMU: value TSS-EM/3Space -> TSS-EM
Routing:
- net 5V: track 240.4 -> 254.4 mm
- net GND: track 188.1 -> 190.1 mm
- net MOTOR: track 74.9 -> 76.3 mm
- net ADC-CON: track 41.3 -> 41.9 mm, vias 1 -> 0
